File: cadeado/Projeto-EEX21-placa/circuito-cadeado/circuito-cadeado.sch (KiCad schematic (older format))
At the start: 15 parts

Commit message: atualização circuito impresso v1.1
Parts:
- added Gnd2, buttom1: 0, Connector_PinSocket_2.54mm:PinSocket_1x02_P2.54mm_Vertical, symbol Connector_Generic:Conn_01x02
- added R4: 10K, Resistor_THT:R_Axial_DIN0204_L3.6mm_D1.6mm_P7.62mm_Horizontal, symbol Device:R
- renumbered Gnd0 to Bateria1
Connections:
- net +9V: now also Bateria1.1 (Pin_1)
- net GNDREF: now also Gnd2.1 (Pin_1), Gnd2.2 (Pin_2), R4.2; no longer Bateria1.1 (Pin_1)
- net at esp1.1 (IO4): no longer servoM1.1 (Pin_1)
- net at esp1.5 (IO13): now also servoM1.1 (Pin_1)
- net at esp1.6 (IO12): now also R4.1, buttom1.1 (Pin_1)
- net at esp1.9 (3V3), mpu6050.8 (Pin_8): now also buttom1.2 (Pin_2)
- no-connect marks 11 -> 10
Other:
- moved on the sheet: Bateria1
Changed lines of the file:
@@
 Wire Wire Line
 	6000 3250 6000 3400
-Wire Wire Line
-	6000 3400 5400 3400
 Connection ~ 5400 3400
 $Comp
@@
 	6200 2850 6100 2850
 Wire Wire Line
-	6100 2850 6100 4200
-Wire Wire Line
 	6100 4200 4600 4200
 Wire Wire Line
@@
 Wire Wire Line
 	4500 4150 4650 4150
-Wire Wire Line
-	4650 4150 4650 3600
 Connection ~ 4650 3400
 Wire Wire Line
@@
 NoConn ~ 7750 2650
 NoConn ~ 7750 3050
-Wire Wire Line
-	6200 2650 6150 2650
-Wire Wire Line
-	6150 2650 6150 3500
 Wire Wire Line
 	6150 3500 7250 3500
@@
 	6950 4100 6950 3350
 Wire Wire Line
-	4400 4100 6950 4100
+	4400 4100 6900 4100
 NoConn ~ 6200 2750
-NoConn ~ 6200 3050
-NoConn ~ 6200 3150
 NoConn ~ 6950 2950
 NoConn ~ 6950 3250
@@
 Connection ~ 4300 2850
 Wire Wire Line
-	4300 2850 4300 2650
+	4300 2850 4300 2800
 Wire Wire Line
 	4300 2900 4300 2850
@@
 	4350 3400 4450 3400
 $Comp
-L Connector_Generic:Conn_01x02 Gnd0
+L Connector_Generic:Conn_01x02 Bateria1
 U 1 1 6198ACB5
-P 5100 3600
-F 0 "Gnd0" V 5064 3412 50  0000 R CNN
-F 1 "0" V 4973 3412 50  0000 R CNN
-F 2 "Connector_PinSocket_2.54mm:PinSocket_1x02_P2.54mm_Vertical" H 5100 3600 50  0001 C CNN
-F 3 "~" H 5100 3600 50  0001 C CNN
-	1    5100 3600
-	1    0    0    -1
-$EndComp
-Connection ~ 4650 3600
-Wire Wire Line
-	4650 3600 4650 3400
+P 4450 3050
+F 0 "Bateria1" V 4414 2862 50  0000 R CNN
+F 1 "0" V 4323 2862 50  0000 R CNN
+F 2 "Connector_PinSocket_2.54mm:PinSocket_1x02_P2.54mm_Vertical" H 4450 3050 50  0001 C CNN
+F 3 "~" H 4450 3050 50  0001 C CNN
+	1    4450 3050
+	1    0    0    -1
+$EndComp
 Wire Wire Line
 	3400 3000 3400 3050
@@
 	4050 3600 4050 3400
 Wire Wire Line
-	4050 3400 4350 3400
+	4050 3400 4250 3400
 Connection ~ 3650 3600
 Wire Wire Line
-	4900 3700 4900 3600
-Connection ~ 4900 3600
-Wire Wire Line
-	4650 3600 4900 3600
-Wire Wire Line
 	3400 3050 3750 3050
+Wire Wire Line
+	4250 3150 4250 3400
+Connection ~ 4250 3400
+Wire Wire Line
+	4250 3400 4350 3400
+Wire Wire Line
+	4250 3050 4200 3050
+Wire Wire Line
+	4200 3050 4200 2800
+Wire Wire Line
+	4200 2800 4300 2800
+Connection ~ 4300 2800
+Wire Wire Line
+	4300 2800 4300 2650
+$Comp
+L Connector_Generic:Conn_01x02 Gnd2
+U 1 1 618CDBE9
+P 4950 3550
+F 0 "Gnd2" V 4914 3362 50  0000 R CNN
+F 1 "0" V 4823 3362 50  0000 R CNN
+F 2 "Connector_PinSocket_2.54mm:PinSocket_1x02_P2.54mm_Vertical" H 4950 3550 50  0001 C CNN
+F 3 "~" H 4950 3550 50  0001 C CNN
+	1    4950 3550
+	1    0    0    -1
+$EndComp
+Wire Wire Line
+	4650 3400 4650 3650
+Wire Wire Line
+	4750 3550 4700 3550
+Wire Wire Line
+	4700 3550 4700 3650
+Wire Wire Line
+	4700 3650 4750 3650
+Wire Wire Line
+	4700 3650 4650 3650
+Connection ~ 4700 3650
+Connection ~ 4650 3650
+Wire Wire Line
+	4650 3650 4650 4150
+Wire Wire Line
+	6100 2850 6100 4200
+Wire Wire Line
+	6150 3500 6150 3050
+Wire Wire Line
+	6150 3050 6200 3050
+NoConn ~ 6200 2650
+$Comp
+L Device:R R4
+U 1 1 618F03C6
+P 6100 4550
+F 0 "R4" H 6170 4596 50  0000 L CNN
+F 1 "10K" H 6170 4505 50  0000 L CNN
+F 2 "Resistor_THT:R_Axial_DIN0204_L3.6mm_D1.6mm_P7.62mm_Horizontal" V 6030 4550 50  0001 C CNN
+F 3 "~" H 6100 4550 50  0001 C CNN
+	1    6100 4550
+	0    1    1    0
+$EndComp
+$Comp
+L Connector_Generic:Conn_01x02 buttom1
+U 1 1 618F353E
+P 6750 4450
+F 0 "buttom1" V 6714 4262 50  0000 R CNN
+F 1 "0" V 6623 4262 50  0000 R CNN
+F 2 "Connector_PinSocket_2.54mm:PinSocket_1x02_P2.54mm_Vertical" H 6750 4450 50  0001 C CNN
+F 3 "~" H 6750 4450 50  0001 C CNN
+	1    6750 4450
+	1    0    0    -1
+$EndComp
+Wire Wire Line
+	7050 4250 6900 4250
+Wire Wire Line
+	6900 4250 6900 4100
+Connection ~ 6900 4100
+Wire Wire Line
+	6900 4100 6950 4100
+Wire Wire Line
+	5400 3400 5700 3400
+Wire Wire Line
+	6200 3150 5950 3150
+Wire Wire Line
+	5950 3150 5950 4450
+Wire Wire Line
+	5950 4450 6300 4450
+Wire Wire Line
+	6300 4450 6300 4550
+Wire Wire Line
+	6300 4550 6250 4550
+Connection ~ 6300 4450
+Wire Wire Line
+	6300 4450 6550 4450
+Wire Wire Line
+	5950 4550 5700 4550
+Wire Wire Line
+	5700 4550 5700 3400
+Connection ~ 5700 3400
+Wire Wire Line
+	5700 3400 6000 3400
+Wire Wire Line
+	6550 4550 6550 4750
+Wire Wire Line
+	6550 4750 7050 4750
+Wire Wire Line
+	7050 4750 7050 4250
 $EndSCHEMATC
